Commit message: metal platform is added

File: husky_description/urdf/husky.urdf.xacro (robot description, xacro)
@@ -1,24 +1,3 @@
 <?xml version="1.0"?>
-<!--
-Software License Agreement (BSD)
-\file      husky.urdf.xacro
-\authors   Paul Bovbel <pbovbel@clearpathrobotics.com>, Devon Ash <dash@clearpathrobotics.com>
-\copyright Copyright (c) 2015, Clearpath Robotics, Inc., All rights reserved.
-Redistribution and use in source and binary forms, with or without modification, are permitted provided that
-the following conditions are met:
- * Redistributions of source code must retain the above copyright notice, this list of conditions and the
-   following disclaimer.
- * Redistributions in binary form must reproduce the above copyright notice, this list of conditions and the
-   following disclaimer in the documentation and/or other materials provided with the distribution.
- * Neither the name of Clearpath Robotics nor the names of its contributors may be used to endorse or promote
-   products derived from this software without specific prior written permission.
-THIS SOFTWARE IS PROVIDED BY THE COPYRIGHT HOLDERS AND CONTRIBUTORS "AS IS" AND ANY EXPRESS OR IMPLIED WAR-
-RANTIES, INCLUDING, BUT NOT LIMITED TO, THE IMPLIED WARRANTIES OF MERCHANTABILITY AND FITNESS FOR A PARTICULAR
-PURPOSE ARE DISCLAIMED. IN NO EVENT SHALL THE COPYRIGHT HOLDER OR CONTRIBUTORS BE LIABLE FOR ANY DIRECT, IN-
-DIRECT, INCIDENTAL, SPECIAL, EXEMPLARY, OR CONSEQUENTIAL DAMAGES (INCLUDING, BUT NOT LIMITED TO, PROCUREMENT
-OF SUBSTITUTE GOODS OR SERVICES; LOSS OF USE, DATA, OR PROFITS; OR BUSINESS INTERRUPTION) HOWEVER CAUSED AND
-ON ANY THEORY OF LIABILITY, WHETHER IN CONTRACT, STRICT LIABILITY, OR TORT (INCLUDING NEGLIGENCE OR OTHERWISE)
-ARISING IN ANY WAY OUT OF THE USE OF THIS SOFTWARE, EVEN IF ADVISED OF THE POSSIBILITY OF SUCH DAMAGE.
--->
 <robot name="husky" xmlns:xacro="http://ros.org/wiki/xacro">
   <!-- IMU Link -->
@@ -40,5 +19,5 @@
   <xacro:arg name="laser_secondary_rpy"     default="$(optenv HUSKY_LMS1XX_SECONDARY_RPY 0.0 0.0 3.14159)" />
   <!-- UST10 Laser Primary  and Secondary -->
-  <xacro:arg name="laser_ust10_front_enabled" default="$(optenv HUSKY_UST10_ENABLED 1)" />
+  <xacro:arg name="laser_ust10_front_enabled" default="$(optenv HUSKY_UST10_ENABLED 0)" />
   <xacro:arg name="laser_ust10_front_topic"   default="$(optenv HUSKY_UST10_TOPIC /scan)" />
   <xacro:arg name="laser_ust10_front_prefix"  default="$(optenv HUSKY_UST10_PREFIX front)" />
@@ -53,11 +32,11 @@
   <xacro:arg name="laser_ust10_rear_rpy"      default="$(optenv HUSKY_UST10_SECONDARY_RPY 0 0 3.14159)" />
   <!-- Velodyne LiDAR Primary and Secondary -->
-  <xacro:arg name="laser_3d_enabled"              default="$(optenv HUSKY_LASER_3D_ENABLED 0)" />
+  <xacro:arg name="laser_3d_enabled"              default="$(optenv HUSKY_LASER_3D_ENABLED 1)" />
   <xacro:arg name="laser_3d_topic"                default="$(optenv HUSKY_LASER_3D_TOPIC points)"/>
   <xacro:arg name="laser_3d_tower"                default="$(optenv HUSKY_LASER_3D_TOWER 1)"/>
   <xacro:arg name="laser_3d_prefix"               default="$(optenv HUSKY_LASER_3D_PREFIX )"/>
-  <xacro:arg name="laser_3d_parent"               default="$(optenv HUSKY_LASER_3D_PARENT top_plate_link)"/>
-  <xacro:arg name="laser_3d_xyz"                  default="$(optenv HUSKY_LASER_3D_XYZ 0 0 0)" />
-  <xacro:arg name="laser_3d_rpy"                  default="$(optenv HUSKY_LASER_3D_RPY 0 0 0)" />
+  <xacro:arg name="laser_3d_parent"               default="$(optenv HUSKY_LASER_3D_PARENT base_link)"/>
+  <xacro:arg name="laser_3d_xyz"                  default="$(optenv HUSKY_LASER_3D_XYZ -0.28513 0 1.1)" />
+  <xacro:arg name="laser_3d_rpy"                  default="$(optenv HUSKY_LASER_3D_RPY 0 0.279253 0)" />
   <xacro:arg name="laser_3d_secondary_enabled"    default="$(optenv HUSKY_LASER_3D_SECONDARY_ENABLED 0)" />
   <xacro:arg name="laser_3d_secondary_topic"      default="$(optenv HUSKY_LASER_3D_SECONDARY_TOPIC secondary_points)"/>
@@ -67,6 +46,6 @@
   <xacro:arg name="laser_3d_secondary_xyz"        default="$(optenv HUSKY_LASER_3D_SECONDARY_XYZ 0 0 0)" />
   <xacro:arg name="laser_3d_secondary_rpy"        default="$(optenv HUSKY_LASER_3D_SECONDARY_RPY 0 0 -3.14159)" />
-  <!-- RealSense Camera Primary and Secondary -->
-  <xacro:arg name="realsense_enabled"             default="$(optenv HUSKY_REALSENSE_ENABLED 1)" />
+  <!-- Realsense Camera Primary and Secondary -->
+  <xacro:arg name="realsense_enabled"             default="$(optenv HUSKY_REALSENSE_ENABLED 0)" />
   <xacro:arg name="realsense_topic"               default="$(optenv HUSKY_REALSENSE_TOPIC realsense)" />
   <xacro:arg name="realsense_prefix"              default="$(optenv HUSKY_REALSENSE_PREFIX camera)" />
@@ -81,5 +60,5 @@
   <xacro:arg name="realsense_secondary_rpy"       default="$(optenv HUSKY_REALSENSE_SECONDARY_RPY 0 0 0)" />
   <!-- BlackflyS Camera Primary and Secondary -->
-  <xacro:arg name="blackfly_enabled"                  default="$(optenv HUSKY_BLACKFLY 1)"/>
+  <xacro:arg name="blackfly_enabled"                  default="$(optenv HUSKY_BLACKFLY 0)"/>
   <xacro:arg name="blackfly_mount_enabled"            default="$(optenv HUSKY_BLACKFLY_MOUNT_ENABLED 1)"/>
   <xacro:arg name="blackfly_mount_angle"              default="$(optenv HUSKY_BLACKFLY_MOUNT_ANGLE 0)"/>
@@ -169,4 +148,116 @@
     <child link="inertial_link" />
   </joint>
+<!-- Metal Platform -->
+<joint name="metal_platform_joint" type="fixed">
+  <parent link="top_plate_front_link"/>
+  <child link="metal_platform_frame"/>
+  <origin xyz="-0.09 0.0 0.18" rpy="0 0 0"/>
+</joint>
+<link name="metal_platform_frame">
+<visual>
+<origin xyz="0.1897 -0.55 -0.267" rpy="0 0 1.57"/>
+<geometry>
+  <mesh filename="package://husky_description/meshes/metal_platform.dae" scale="0.001 0.001 0.001" />
+</geometry>
+</visual>
+<collision>
+<origin xyz="0.1897 -0.55 -0.267" rpy="0 0 1.57"/>
+<geometry>
+  <mesh filename="package://husky_description/meshes/metal_platform.STL" scale="0.001 0.001 0.001"/>
+</geometry>
+</collision>
+</link>
+<!-- Boxe_1 -->
+<joint name="Boxe_1_joint" type="fixed">
+        <parent link="base_link"/>
+        <child link="Boxe_1_frame"/>
+        <origin xyz="-0.28 0 1.155" rpy="0 0 0"/>
+    </joint>
+ <link name="Boxe_1_frame">
+   <visual>
+     <origin xyz="0 0 0" rpy="0 0 0" />
+     <geometry>
+       <box size="0.04 0.52 0.01" />
+     </geometry>
+     <material name="grey" >
+    <color rgba="0.5725490196078431 0.5843137254901961 0.5686274509803921 1.0" />
+     </material>
+   </visual>
+   <collision>
+     <origin xyz="0 0 0" rpy="0 0 0"/>
+     <geometry>
+        <box size="0.04 0.52 0.01" />
+     </geometry>
+   </collision>
+ </link>
+<!-- Boxe_2 -->
+<joint name="Boxe_2_joint" type="fixed">
+        <parent link="base_link"/>
+        <child link="Boxe_2_frame"/>
+        <origin xyz="-0.28 0.26 0.703" rpy="0 0 0"/>
+    </joint>
+ <link name="Boxe_2_frame">
+   <visual>
+     <origin xyz="0 0 0" rpy="0 0 0"/>
+     <geometry>
+       <box size="0.04 0.01 0.904" />
+     </geometry>
+     <material name="grey" >
+    <color rgba="0.8 0.8 0.8 1.0" />
+     </material>
+   </visual>
+   <collision>
+    <origin xyz="0 0 0" rpy="0 0 0"/>
+     <geometry>
+        <box size="0.04 0.01 0.904" />
+     </geometry>
+   </collision>
+ </link>
+<!-- Boxe_3 -->
+<joint name="Boxe_3_joint" type="fixed">
+        <parent link="base_link"/>
+        <child link="Boxe_3_frame"/>
+        <origin xyz="-0.28 -0.26 0.703" rpy="0 0 0"/>
+    </joint>
+ <link name="Boxe_3_frame">
+   <visual>
+     <origin xyz="0 0 0" rpy="0 0 0"/>
+     <geometry>
+       <box size="0.04 0.01 0.904" />
+     </geometry>
+     <material name="grey" >
+    <color rgba="0.8 0.8 0.8 1.0" />
+     </material>
+   </visual>
+   <collision>
+    <origin xyz="0 0 0" rpy="0 0 0"/>
+     <geometry>
+        <box size="0.04 0.01 0.904" />
+     </geometry>
+   </collision>
+ </link>
+ <!-- RTK -->
+<joint name="rtk_joint" type="fixed">
+        <parent link="base_link"/>
+        <child link="rtk_frame"/>
+        <origin xyz="-0.28 0.21 1.16" rpy="0 0 0"/>
+    </joint>
+ <link name="rtk_frame">
+   <visual>
+     <origin xyz="0 0 0" rpy="0 0 0"/>
+     <geometry>
+        <cylinder radius="0.01" length="0.01"/>
+     </geometry>
+     <material name="black" >
+    <color rgba="0 0 0 1.0" />
+     </material>
+   </visual>
+   <collision>
+    <origin xyz="0 0 0" rpy="0 0 0"/>
+     <geometry>
+        <cylinder radius="0.01" length="0.01"/>
+     </geometry>
+   </collision>
+ </link>
   <!-- Husky wheel macros -->
   <xacro:husky_wheel wheel_prefix="front_left">
